File: Electronics/OpenThereminV4.kicad_sch (KiCad schematic)
At the start: 104 parts, among them J1 USB_C_Receptacle, J2 Conn_02x03_Odd_Even, P1 10k, P10 BUTTON, P11 A3_PAD, P12 A2_PAD, P13 A1_PAD, P14 A0_PAD, P15 CV2, P16 GND, P2 10k, P3 10k, P4 10k, P5 VCC, P6 audio, P7 CV1, P8 VCC, P9 GND, U1 TTP223, U10 CH340G, U11 LP2985-3.3, U12 MCP4922-E/SL, U2 4060, U3 4060, U4 74HC74, U5 4069, U6 MCP4921-E/SN, U7 MCP4922-E/SL, U8 LM358 / MCP6002, U9 ATmega328P-AU, X1 16MHz, X2 7.3721MHz, X3 12MHz, Y1 MountPad3, Y2 MountPad3, Y3 PLUG_3_5_SMD, Y7 PLUG_3_5_SMD

Commit message: clean design, updates
Parts:
- removed U6: MCP4921-E/SN, Package_SO:SOIC-8_3.9x4.9mm_P1.27mm, symbol OpenThereminV4-rescue:MCP4921-E_SN
- added U6: MCP4922-E/SL, Package_SO:SOIC-14_3.9x8.7mm_P1.27mm, symbol OpenThereminV4-rescue:MCP4922-E_SL
- J2, P10, P11, P12, P13, P14, P15, P16, P6, P7, P8, P9: now left out of the parts list
- P5: value VCC -> RXD; now left out of the parts list
- W1, W2: footprint GaudiLabsFootPrints:Fiducial_1mm_Dia_2.54mm_Outer_CopperBottom -> Fiducial:Fiducial_1mm_Mask2mm; now left out of the parts list
Connections:
- net DAC_CS: now also U6.3 (~{CS})
- net DAC_DI: now also U6.5 (SDI)
- net DAC_LATCH: now also U6.8 (~{LDAC})
- net DAC_SCK: now also U6.4 (SCK)
- net GND: now also J1.S1 (SHIELD), U6.12 (AVSS)
- net VCC: now also U6.1 (VDD), U6.9 (~{SHDN})
- net VREF: now also U6.11 (VrefB), U6.13 (VrefA)
- net at R17.1: now also U6.14 (VoutA)
Other:
- moved on the sheet: C21, R16, R17

Commit message: label update
Parts:
- ?: footprint GaudiLabsFootPrints:GNDPad -> MountingHole:MountingHole_3mm_Pad_Via
Connections:
- net at C11.1, C12.1, C9.1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: no longer C10.1, C9.2, R5.2, U5.5
- net at C2.1, C4.1, C5.1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: no longer C2.2, C3.1, R1.2, U5.9
- new net: C10.1, C9.2, R5.2, U5.5
- new net: C2.2, C3.1, R1.2, U5.9
Changed lines of the file:
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@@
   (junction (at 234.95 43.18) (diameter 0) (color 0 0 0 0)
   )
-  (junction (at 44.45 133.35) (diameter 0) (color 0 0 0 0)
-  )
   (junction (at 232.41 43.18) (diameter 0) (color 0 0 0 0)
   )
@@
   (junction (at 26.67 90.17) (diameter 0) (color 0 0 0 0)
   )
-  (junction (at 44.45 45.72) (diameter 0) (color 0 0 0 0)
-  )
   (junction (at 92.71 172.72) (diameter 0) (color 0 0 0 0)
   )
@@
     (stroke (width 0) (type default) (color 0 0 0 0))
   )
-  (wire (pts (xy 44.45 144.78) (xy 44.45 133.35))
-    (stroke (width 0) (type default) (color 0 0 0 0))
-  )
   (wire (pts (xy 204.47 41.91) (xy 204.47 44.45))
     (stroke (width 0) (type default) (color 0 0 0 0))
@@
     (stroke (width 0) (type default) (color 0 0 0 0))
   )
-  (wire (pts (xy 44.45 144.78) (xy 39.37 144.78))
+  (wire (pts (xy 43.18 144.78) (xy 39.37 144.78))
     (stroke (width 0) (type default) (color 0 0 0 0))
   )
@@
     (stroke (width 0) (type default) (color 0 0 0 0))
   )
-  (wire (pts (xy 44.45 43.18) (xy 40.64 43.18))
+  (wire (pts (xy 43.18 43.18) (xy 40.64 43.18))
     (stroke (width 0) (type default) (color 0 0 0 0))
   )
@@
     (stroke (width 0) (type default) (color 0 0 0 0))
   )
-  (wire (pts (xy 44.45 133.35) (xy 44.45 130.81))
-    (stroke (width 0) (type default) (color 0 0 0 0))
-  )
   (wire (pts (xy 64.77 115.57) (xy 69.85 115.57))
     (stroke (width 0) (type default) (color 0 0 0 0))
@@
     (stroke (width 0) (type default) (color 0 0 0 0))
   )
-  (wire (pts (xy 44.45 45.72) (xy 44.45 43.18))
+  (wire (pts (xy 43.18 43.18) (xy 43.18 57.15))
     (stroke (width 0) (type default) (color 0 0 0 0))
   )
@@
     (stroke (width 0) (type default) (color 0 0 0 0))
   )
+  (wire (pts (xy 43.18 130.81) (xy 40.64 130.81))
+    (stroke (width 0) (type default) (color 0 0 0 0))
+  )
   (wire (pts (xy 170.18 262.89) (xy 171.45 262.89))
     (stroke (width 0) (type default) (color 0 0 0 0))
@@
     (stroke (width 0) (type default) (color 0 0 0 0))
   )
-  (wire (pts (xy 44.45 57.15) (xy 44.45 45.72))
-    (stroke (width 0) (type default) (color 0 0 0 0))
-  )
   (wire (pts (xy 304.8 135.89) (xy 304.8 138.43))
     (stroke (width 0) (type default) (color 0 0 0 0))
@@
     (stroke (width 0) (type default) (color 0 0 0 0))
   )
-  (wire (pts (xy 44.45 130.81) (xy 40.64 130.81))
-    (stroke (width 0) (type default) (color 0 0 0 0))
-  )
   (wire (pts (xy 354.33 78.74) (xy 349.25 78.74))
     (stroke (width 0) (type default) (color 0 0 0 0))
@@
     (stroke (width 0) (type default) (color 0 0 0 0))
   )
-  (wire (pts (xy 44.45 57.15) (xy 39.37 57.15))
+  (wire (pts (xy 43.18 57.15) (xy 39.37 57.15))
     (stroke (width 0) (type default) (color 0 0 0 0))
   )
@@
     (stroke (width 0) (type default) (color 0 0 0 0))
   )
+  (wire (pts (xy 43.18 130.81) (xy 43.18 144.78))
+    (stroke (width 0) (type default) (color 0 0 0 0))
+  )
   (wire (pts (xy 40.64 107.95) (xy 40.64 115.57))
     (stroke (width 0) (type default) (color 0 0 0 0))
@@
   (symbol (lib_id "OpenThereminV4-rescue:4069") (at 52.07 115.57 0) (unit 3)
     (in_bom yes) (on_board yes)
-    (property "Reference" "U5" (id 0) (at 52.07 107.569 0))
+    (property "Reference" "U5" (id 0) (at 54.61 119.38 0))
     (property "Value" "4069" (id 1) (at 52.07 109.8804 0))
     (property "Footprint" "Package_SO:SOIC-14_3.9x8.7mm_P1.27mm" (id 2) (at 52.07 115.57 0)
@@
   (symbol (lib_id "OpenThereminV4-rescue:TEST_1P") (at 76.2 180.34 0) (unit 1)
     (in_bom yes) (on_board yes)
-    (property "Reference" "" (id 0) (at 74.93 176.53 0)
+    (property "Reference" "" (id 0) (at 78.74 175.26 0)
       (effects (font (size 1.27 1.27)) (justify right))
     )
@@
       (effects (font (size 1.27 1.27)) (justify right))
     )
-    (property "Footprint" "GaudiLabsFootPrints:GNDPad" (id 2) (at 81.28 180.34 0)
+    (property "Footprint" "MountingHole:MountingHole_3mm_Pad_Via" (id 2) (at 81.28 180.34 0)
       (effects (font (size 1.27 1.27)) hide)
     )
@@
     )
     (path "/00000000-0000-0000-0000-00005735d84b"
-      (reference "GROUND1") (unit 1) (value "GND_PAD") (footprint "GaudiLabsFootPrints:GNDPad")
+      (reference "GND1") (unit 1) (value "GND_PAD") (footprint "MountingHole:MountingHole_3mm_Pad_Via")
     )
     (path "/00000000-0000-0000-0000-0000605d6c3e"

Commit message: update kicad files
Parts:
- removed C19, C31: 33pF, Capacitor_SMD:C_0603_1608Metric, symbol OpenThereminV4-rescue:C
- removed R10, R9: 2.2k, Resistor_SMD:R_0603_1608Metric, symbol OpenThereminV4-rescue:RES
- removed U10: CH340G, Package_SO:SOIC-16_3.9x9.9mm_P1.27mm, symbol Interface_USB:CH340G
- removed X3: 12MHz, Crystal:Crystal_SMD_HC49-SD, symbol OpenThereminV4-rescue:Crystal_Small
- added D4: DualLED, Mlab_D:LED_DUAL_WL-SBRW, symbol OpenThereminV4-rescue:DualLED-GaudiLabsPartsLibrary
- added R23, R24: 470R, Resistor_SMD:R_0603_1608Metric, symbol OpenThereminV4-rescue:RES
- added U10: FT232RL, Package_SO:SSOP-28_5.3x10.2mm_P0.65mm, symbol Interface_USB:FT232RL
- C1: value 220pF -> 150pF NP0; mouser (none) -> OK NPO
- C10, C2, C3, C9: value 150pF -> 150pF NP0; mouser (none) -> OK NPO
- C11: value 10pF -> 10pF NP0; mouser (none) -> OK NPO
- C12, C5: value 470pF -> 470pF NP0; mouser (none) -> OK NPO
- C13, C23, C24, C25, C26, C27, C28, C29, C6, D1, D2, R15, R16, R3, R4, R7, R8, U11, U4, U8, X1, Y1, Y2: mouser (none) -> OK
- C14: value not assembled -> 47pF NP0; mouser (none) -> OK NPO
- C15, C16, C17, C18: value 33pF -> 22pF; mouser (none) -> OK
- C20, C21, C30, C32, C33, C35: value 100n -> 100nF; mouser (none) -> OK
- C22: value 10n -> 10nF; mouser (none) -> OK
- C34: value 22n -> 22nF; mouser (none) -> OK
- C36: value 47u -> 47uF; mouser (none) -> OK
- C37: value 1u -> 1uF; mouser (none) -> OK
- C4, J2, P10, W1, W2: mouser (none) -> -
- C7: value not assembled -> 150pF NP0; mouser (none) -> OK NPO
- C8: value 330pF -> 150pF NP0; mouser (none) -> OK NPO
- D3: footprint GaudiLabsFootPrints:WL-SBRW -> Mlab_D:LED_DUAL_WL-SBRW; mouser (none) -> OK
- GND1: renamed from ?; mouser (none) -> -
- J1: footprint GaudiLabsFootPrints:USB_C_Receptacle_Amphenol_12401610E4-2A -> Mlab_CON:USBC GCT_USB4105-GF-A; symbol OpenThereminV4-rescue:USB_C_Receptacle-GaudiLabsPartsLibrary -> Connector:USB_C_Receptacle_USB2.0; mouser (none) -> OK
- L1: footprint Inductor_SMD:L_1008_2520Metric -> Inductor_SMD:L_1812_4532Metric; MFNP (none) -> CC453232A-102KL; mouser (none) -> OK
- L2: footprint GaudiLabsFootPrints:COIL -> Inductor_SMD:L_1812_4532Metric; MFNP (none) -> CC453232A-102KL; mouser (none) -> OK
- P1, P2, P3, P4: MFNP (none) -> PS15NV60; mouser (none) -> OK
- P11, P12, P13, P14, P15, P16, P5, P6, P7, P8, P9: footprint GaudiLabsFootPrints:SMD_Pinheader_1_OT_BLANK -> TestPoint:TestPoint_Pad_1.5x1.5mm; mouser (none) -> -
- R1, R11, R13, R5: value 4.7M -> 4M7; mouser (none) -> OK
- R12, R14, R18, R19: value 470 -> 470R; mouser (none) -> OK
- R17, R2, R20, R21, R22, R6: value 2.2k -> 2k2; mouser (none) -> OK
- U1: mouser (none) -> dratek/dis
- U12, U6, U7, U9: mouser (none) -> LCSC
- U2, U3: value 4060 -> 74HC4060D; mouser (none) -> OK
- U5: value 4069 -> HEF4069UBT; mouser (none) -> OK
- X2: mouser (none) -> Ok
- Y3, Y7: value PLUG_3_5_SMD -> SJ-3524-SMT-TR; footprint GaudiLabsFootPrints:SJ-3502-SMT-TR -> Connector_Audio:Jack_3.5mm_CUI_SJ-3524-SMT_Horizontal; symbol OpenThereminV4-rescue:PLUG_3_5_SMD -> Connector:AudioJack3; mouser (none) -> OK
Connections:
- net D+: now also U10.15 (USBD+)
- net D-: now also U10.16 (USBD-)
- net GND: now also Y3.S, Y7.S, D4.1, D4.2, U10.18 (GND), U10.21 (GND), U10.25 (AGND), U10.7 (GND); no longer Y3.1 (GND), Y7.1 (GND)
- net RXD: now also U10.5 (RXD)
- net TXD: now also U10.1 (TXD)
- net VCC: now also U10.19 (~{RESET}), U10.20 (VCC), U10.4 (VCCIO)
- net at C29.2, P6.1 (P1): now also Y7.R, Y7.T; no longer Y7.3 (L)
- net at P15.1 (P1), U12.10 (VoutB): now also Y3.T; no longer Y3.2 (R)
- net at P7.1 (P1), U12.14 (VoutA): now also Y3.R; no longer Y3.3 (L)
- net at C32.2: now also U10.2 (DTR)
- net at C30.1: now also U10.17 (3V3OUT)
- new net: D4.3, R24.1
- new net: R24.2, U10.23 (CBUS0)
- new net: R23.2, U10.22 (CBUS1)
- new net: D4.4, R23.1
Other:
- moved on the sheet: C30, C32, P16, P7
