File: Electronics/OpenThereminV4.kicad_sch (KiCad schematic)
At the start: 102 parts, among them J1 USB_C_Receptacle, J2 Conn_02x03_Odd_Even, P1 10k, P10 BUTTON, P11 A3_PAD, P12 A2_PAD, P13 A1_PAD, P14 A0_PAD, P15 CV2, P16 GND, P2 10k, P3 10k, P4 10k, P5 RXD, P6 audio, P7 CV1, P8 VCC, P9 GND, U1 TTP223, U10 FT232RL, U11 LP2985-3.3, U12 MCP4922-E/SL, U2 74HC4060D, U3 74HC4060D, U4 74HC74, U5 HEF4069UBT, U6 MCP4922-E/SL, U7 MCP4922-E/SL, U8 LM358 / MCP6002, U9 ATmega328P-AU, X1 16MHz, X2 7.3721MHz, Y1 MountPad3, Y2 MountPad3, Y3 SJ-3524-SMT-TR, Y7 SJ-3524-SMT-TR

Commit message: update files
Connections:
- no-connect marks 0 -> 41
Changed lines of the file:
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@@
   (junction (at 33.02 135.89) (diameter 0) (color 0 0 0 0)
   )
+  (no_connect (at 245.11 219.71))
+  (no_connect (at 120.65 33.02))
+  (no_connect (at 154.94 193.04))
+  (no_connect (at 120.65 120.65))
+  (no_connect (at 146.05 27.94))
+  (no_connect (at 146.05 138.43))
+  (no_connect (at 318.77 63.5))
+  (no_connect (at 146.05 45.72))
+  (no_connect (at 146.05 33.02))
+  (no_connect (at 146.05 38.1))
+  (no_connect (at 157.48 223.52))
+  (no_connect (at 245.11 234.95))
+  (no_connect (at 146.05 125.73))
+  (no_connect (at 204.47 240.03))
+  (no_connect (at 146.05 130.81))
+  (no_connect (at 245.11 212.09))
+  (no_connect (at 146.05 50.8))
+  (no_connect (at 349.25 73.66))
+  (no_connect (at 245.11 209.55))
+  (no_connect (at 146.05 48.26))
+  (no_connect (at 320.04 201.93))
+  (no_connect (at 245.11 240.03))
+  (no_connect (at 204.47 227.33))
+  (no_connect (at 146.05 118.11))
+  (no_connect (at 245.11 217.17))
+  (no_connect (at 146.05 43.18))
+  (no_connect (at 199.39 36.83))
+  (no_connect (at 182.88 77.47))
+  (no_connect (at 320.04 199.39))
+  (no_connect (at 149.86 193.04))
+  (no_connect (at 245.11 222.25))
+  (no_connect (at 146.05 120.65))
+  (no_connect (at 228.6 99.06))
+  (no_connect (at 204.47 232.41))
+  (no_connect (at 146.05 133.35))
+  (no_connect (at 146.05 123.19))
+  (no_connect (at 146.05 135.89))
+  (no_connect (at 245.11 237.49))
+  (no_connect (at 182.88 111.76))
+  (no_connect (at 146.05 128.27))
+  (no_connect (at 146.05 35.56))
   (wire (pts (xy 354.33 55.88) (xy 349.25 55.88))
     (stroke (width 0) (type default) (color 0 0 0 0))
@@
     (effects (font (size 1.524 1.524)) (justify left bottom))
   )
-  (label "JMP" (at 292.1 46.99 0)
+  (label "JMP" (at 289.56 46.99 0)
     (effects (font (size 1.524 1.524)) (justify left bottom))
   )

Commit message: update bom
Parts:
- U12, U6, U7: mouser LCSC -> OK
Changed lines of the file:
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@@
     )
     (property "Datasheet" "" (id 3) (at 76.2 85.09 0))
-    (property "mouser" "LCSC" (id 4) (at 76.2 85.09 0)
+    (property "mouser" "OK" (id 4) (at 76.2 85.09 0)
       (effects (font (size 1.27 1.27)) hide)
     )
@@
     )
     (property "Datasheet" "" (id 3) (at 243.84 93.98 0))
-    (property "mouser" "LCSC" (id 4) (at 243.84 93.98 0)
+    (property "mouser" "OK" (id 4) (at 243.84 93.98 0)
       (effects (font (size 1.27 1.27)) hide)
     )
@@
     )
     (property "Datasheet" "" (id 3) (at 184.15 31.75 0))
-    (property "mouser" "LCSC" (id 4) (at 184.15 31.75 0)
-      (effects (font (size 1.27 1.27)) hide)
-    )
+    (property "mouser" "OK" (id 4) (at 184.15 31.75 0)
+      (effects (font (size 1.27 1.27)) hide)
+    )
