File: Electronics/OpenThereminV4.kicad_pcb (KiCad board)
At the start: 2 copper layers, 50.5 x 127.5 mm, 110 parts, among them J1 USB_C_Receptacle, J2 Conn_02x03_Odd_Even, P1 10k, P10 BUTTON, P11 A3_PAD, P12 A2_PAD, P13 A1_PAD, P14 A0_PAD, P15 CV2, P16 GND, P2 10k, P3 10k, P4 10k, P5 VCC, P6 audio, P7 CV1, P8 VCC, P9 GND, U1 TTP223, U10 CH340G, U11 LP2985-3.3, U12 MCP4922-E/SL, U2 4060, U3 4060, U4 74HC74, U5 4069, U6 MCP4921-E/SN, U7 MCP4922-E/SL, U8 LM358 / MCP6002, U9 ATmega328P-AU, X1 16MHz, X2 7.3721MHz, X3 12MHz, Y1 MountPad3, Y2 MountPad3, Y3 PLUG_3_5_SMD, Y7 PLUG_3_5_SMD

Commit message: clean kicad files, update to kicad v6
Other:
- net class Default removed
- net class FAT removed
- net class Power removed
- net class Thin removed

Commit message: clean design, updates
Parts:
- removed G***: LOGO, GaudiLabsLogos:OpenHardware_gold
- removed G***: LOGO, GaudiLabsLogos:OT_credits
- removed G***: LOGO, GaudiLabsLogos:Peace_logo
- removed G***: LOGO, GaudiLabsLogos:OT_gold_logo
- removed G***: LOGO, GaudiLabsLogos:OT_gold_gnd
- removed G***: LOGO, GaudiLabsLogos:OSHW_OT3
- P5: value VCC -> RXD
- U6: value MCP4921-E/SN -> MCP4922-E/SL; footprint Package_SO:SOIC-8_3.9x4.9mm_P1.27mm -> Package_SO:SOIC-14_3.9x8.7mm_P1.27mm
- W1, W2: footprint GaudiLabsFootPrints:Fiducial_1mm_Dia_2.54mm_Outer_CopperBottom -> Fiducial:Fiducial_1mm_Mask2mm
- moved C24 4.18 mm to (93.5, 146.0)
- moved C21 2.35 mm to (94.8, 141.6)
- moved R16 1.46 mm to (95.7, 143.1)
- moved U3 0.94 mm to (88.2, 139.0)
- moved U6 0.89 mm to (97.8, 136.1), turned to 180 degrees
- moved U2 0.52 mm to (80.3, 138.2)
- moved R13 0.28 mm to (90.7, 145.5)
- moved R14 0.28 mm to (90.7, 147.0)
- moved C30 0.14 mm to (101.1, 113.6)
- turned R19 to 0 degrees
Connections:
- C11 pad 1: Net-(C11-Pad1) -> Net-(C10-Pad1)
- C12 pad 1: Net-(C11-Pad1) -> Net-(C10-Pad1)
- C2 pad 2: Net-(C2-Pad2) -> Net-(C2-Pad1)
- C3 pad 1: Net-(C2-Pad2) -> Net-(C2-Pad1)
- C9 pad 1: Net-(C11-Pad1) -> Net-(C10-Pad1)
- J1 pad A10: (no net) -> unconnected-(J1-PadA10)
- J1 pad A11: (no net) -> unconnected-(J1-PadA11)
- J1 pad A2: (no net) -> unconnected-(J1-PadA2)
- J1 pad A3: (no net) -> unconnected-(J1-PadA3)
- J1 pad A8: (no net) -> unconnected-(J1-PadA8)
- J1 pad B10: (no net) -> unconnected-(J1-PadB10)
- J1 pad B11: (no net) -> unconnected-(J1-PadB11)
- J1 pad B2: (no net) -> unconnected-(J1-PadB2)
- J1 pad B3: (no net) -> unconnected-(J1-PadB3)
- J1 pad B8: (no net) -> unconnected-(J1-PadB8)
- J1 pad S1: Net-(J1-PadS1) -> GND
- L2 pad 1: Net-(C11-Pad1) -> Net-(C10-Pad1)
- R1 pad 2: Net-(C2-Pad2) -> Net-(C2-Pad1)
- U10 pad 10: (no net) -> unconnected-(U10-Pad10)
- U10 pad 11: (no net) -> unconnected-(U10-Pad11)
- U10 pad 12: (no net) -> unconnected-(U10-Pad12)
- U10 pad 14: (no net) -> unconnected-(U10-Pad14)
- U10 pad 15: (no net) -> unconnected-(U10-Pad15)
- U10 pad 9: (no net) -> unconnected-(U10-Pad9)
- U11 pad 4: (no net) -> unconnected-(U11-Pad4)
- U12 pad 9: (no net) -> unconnected-(U12-Pad9)
- U2 pad 1: (no net) -> unconnected-(U2-Pad1)
- U2 pad 14: (no net) -> unconnected-(U2-Pad14)
- U2 pad 15: (no net) -> unconnected-(U2-Pad15)
- U2 pad 2: (no net) -> unconnected-(U2-Pad2)
- U2 pad 3: (no net) -> unconnected-(U2-Pad3)
- U2 pad 4: (no net) -> unconnected-(U2-Pad4)
- U2 pad 6: (no net) -> unconnected-(U2-Pad6)
- U2 pad 7: (no net) -> unconnected-(U2-Pad7)
- U2 pad 9: (no net) -> unconnected-(U2-Pad9)
- U3 pad 1: (no net) -> unconnected-(U3-Pad1)
- U3 pad 13: (no net) -> unconnected-(U3-Pad13)
- U3 pad 14: (no net) -> unconnected-(U3-Pad14)
- U3 pad 15: (no net) -> unconnected-(U3-Pad15)
- U3 pad 2: (no net) -> unconnected-(U3-Pad2)
- U3 pad 3: (no net) -> unconnected-(U3-Pad3)
- U3 pad 4: (no net) -> unconnected-(U3-Pad4)
- U3 pad 5: (no net) -> unconnected-(U3-Pad5)
- U3 pad 6: (no net) -> unconnected-(U3-Pad6)
- U3 pad 9: (no net) -> unconnected-(U3-Pad9)
- U4 pad 6: (no net) -> unconnected-(U4-Pad6)
- U4 pad 8: (no net) -> unconnected-(U4-Pad8)
- U5 pad 9: Net-(C2-Pad2) -> Net-(C2-Pad1)
- U6 pad 2: DAC_CS -> (no net)
- U6 pad 3: DAC_SCK -> DAC_CS
- U6 pad 4: DAC_DI -> DAC_SCK
- U6 pad 5: DAC_LATCH -> DAC_DI
- U6 pad 6: VREF -> (no net)
- U6 pad 7: GND -> (no net)
- U6 pad 8: Net-(R17-Pad1) -> DAC_LATCH
- U9 pad 22: (no net) -> unconnected-(U9-Pad22)
- U9 pad 8: (no net) -> unconnected-(U9-Pad8)
- Y2 pad 1: Net-(C11-Pad1) -> Net-(C10-Pad1)
- Y7 pad 2: (no net) -> unconnected-(Y7-Pad2)
Routing:
- net GND: track 127.3 -> 59.2 mm, vias 35 -> 44
- net Net-(C11-Pad1): track 47.6 -> 0.00 mm
- net Net-(C10-Pad1): track 26.2 -> 73.5 mm
- net Net-(C2-Pad2): track 27.9 -> 0.00 mm
- net Net-(C2-Pad1): track 43.4 -> 70.2 mm
- net VREF: track 16.8 -> 24.7 mm
- net Net-(R17-Pad1): track 17.1 -> 24.9 mm
- net LED_RED: track 33.4 -> 25.8 mm
- net DAC_DI: track 60.9 -> 54.9 mm
- net VCC: track 309.6 -> 314.6 mm, vias 24 -> 25
- net DAC_LATCH: track 60.8 -> 55.8 mm
- net VO_PITCH: track 64.9 -> 60.6 mm
- net Net-(U3-Pad7): track 45.1 -> 41.7 mm
- net DAC_SCK: track 71.5 -> 68.3 mm
- net VO_VOL: track 61.0 -> 58.0 mm
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Other:
- board text added: "OpenTheremin V4"
- board text removed: "4060"
- board text removed: "4069"
- board text removed: "7474"
- board text removed: "MCP4921"
- board text removed: "MCP4922"
- board text removed: "MCP6002"
- board text removed: "V3.0 2016"
- board text removed: "gaudi.ch"

Commit message: label update
Parts:
- removed GROUND1: GND_PAD, GaudiLabsFootPrints:GNDPad
- added GND1: GND_PAD, MountingHole:MountingHole_3mm_Pad_Via, F.Cu at (79.8, 148.3)
- moved C17 4.58 mm to (103.8, 154.6), turned to -90 degrees
- moved C18 1.16 mm to (114.0, 151.6), turned to 0 degrees
Connections:
- C10 pad 1: Net-(C10-Pad1) -> Net-(R5-Pad2)
- C11 pad 1: Net-(C10-Pad1) -> Net-(C11-Pad1)
- C12 pad 1: Net-(C10-Pad1) -> Net-(C11-Pad1)
- C2 pad 2: Net-(C2-Pad1) -> Net-(C2-Pad2)
- C3 pad 1: Net-(C2-Pad1) -> Net-(C2-Pad2)
- C9 pad 1: Net-(C10-Pad1) -> Net-(C11-Pad1)
- C9 pad 2: Net-(C10-Pad1) -> Net-(R5-Pad2)
- L2 pad 1: Net-(C10-Pad1) -> Net-(C11-Pad1)
- R1 pad 2: Net-(C2-Pad1) -> Net-(C2-Pad2)
- R5 pad 2: Net-(C10-Pad1) -> Net-(R5-Pad2)
- U5 pad 5: Net-(C10-Pad1) -> Net-(R5-Pad2)
- U5 pad 9: Net-(C2-Pad1) -> Net-(C2-Pad2)
- Y2 pad 1: Net-(C10-Pad1) -> Net-(C11-Pad1)
Routing:
- net Net-(C10-Pad1): track 73.5 -> 0.00 mm
- net Net-(C11-Pad1): track 0.00 -> 46.7 mm
- net Net-(C2-Pad1): track 70.2 -> 43.4 mm
- net Net-(R5-Pad2): track 0.00 -> 25.6 mm
- net Net-(C2-Pad2): track 0.00 -> 25.6 mm
- net GND: track 59.2 -> 46.7 mm, vias 44 -> 53
- net Net-(C34-Pad1): track 20.4 -> 8.18 mm
- net Net-(U12-Pad14): track 41.9 -> 35.7 mm
- net Net-(C18-Pad1): track 35.9 -> 30.0 mm
- net Net-(U3-Pad11): track 35.2 -> 30.3 mm
- net Net-(Y7-Pad3): track 16.5 -> 13.6 mm
- net VCC: track 314.6 -> 312.5 mm
- net Net-(C22-Pad1): track 13.2 -> 11.5 mm
- net A3: track 51.7 -> 50.1 mm
- net Net-(J1-PadA5): track 15.3 -> 14.3 mm
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- added copper zone on F.Cu, net Net-(U12-Pad10)
- added copper zone on B.Cu, net Net-(U12-Pad14)
- added copper zone on B.Cu, net Net-(Y7-Pad3)
- added copper zone on F.Cu, net unconnected-(Y7-Pad2)
Other:
- board text added: "CV"
- board text added: "Function"
- board text added: "Ground"
- board text added: "Out"
- board text added: "Pitch"
- board text added: "Register"
- board text added: "Timber"
- board text added: "USB-C"
- board text added: "Volume"
- board text removed: "back"
- board text removed: "front"

Commit message: update kicad files
Parts:
- removed C19, C31: 33pF, Capacitor_SMD:C_0603_1608Metric
- removed R10, R9: 2.2k, Resistor_SMD:R_0603_1608Metric
- removed X3: 12MHz, Crystal:Crystal_SMD_HC49-SD
- added D4: DualLED, Mlab_D:LED_DUAL_WL-SBRW, B.Cu at (100.0, 100.8)
- added R23: 470R, Resistor_SMD:R_0603_1608Metric, B.Cu at (99.3, 105.0)
- added R24: 470R, Resistor_SMD:R_0603_1608Metric, B.Cu at (100.9, 105.0)
- C1: value 220pF -> 150pF NP0
- C10, C2, C3, C9: value 150pF -> 150pF NP0
- C11: value 10pF -> 10pF NP0
- C12, C5: value 470pF -> 470pF NP0
- C14: value not assembled -> 47pF NP0
- C15, C16, C17, C18: value 33pF -> 22pF
- C20, C21, C30, C32, C33, C35: value 100n -> 100nF
- C22: value 10n -> 10nF
- C34: value 22n -> 22nF
- C36: value 47u -> 47uF
- C37: value 1u -> 1uF
- C7: value not assembled -> 150pF NP0
- C8: value 330pF -> 150pF NP0
- D3: footprint GaudiLabsFootPrints:WL-SBRW -> Mlab_D:LED_DUAL_WL-SBRW
- J1: footprint GaudiLabsFootPrints:USB_C_Receptacle_Amphenol_12401610E4-2A -> Mlab_CON:USBC GCT_USB4105-GF-A
- L1: footprint Inductor_SMD:L_1008_2520Metric -> Inductor_SMD:L_1812_4532Metric
- L2: footprint GaudiLabsFootPrints:COIL -> Inductor_SMD:L_1812_4532Metric
- P11, P12, P13, P14, P15, P16, P5, P6, P7, P8, P9: footprint GaudiLabsFootPrints:SMD_Pinheader_1_OT_BLANK -> TestPoint:TestPoint_Pad_1.5x1.5mm
- R1, R11, R13, R5: value 4.7M -> 4M7
- R12, R14, R18, R19: value 470 -> 470R
- R17, R2, R20, R21, R22, R6: value 2.2k -> 2k2
- U10: value CH340G -> FT232RL; footprint Package_SO:SOIC-16_3.9x9.9mm_P1.27mm -> Package_SO:SSOP-28_5.3x10.2mm_P0.65mm
- U2, U3: value 4060 -> 74HC4060D
- U5: value 4069 -> HEF4069UBT
- Y3, Y7: value PLUG_3_5_SMD -> SJ-3524-SMT-TR; footprint GaudiLabsFootPrints:SJ-3502-SMT-TR -> Connector_Audio:Jack_3.5mm_CUI_SJ-3524-SMT_Horizontal
- moved C30 14.8 mm to (115.3, 117.9), turned to -90 degrees
- moved C18 11.9 mm to (102.3, 153.4), turned to -90 degrees
- moved Y7 6.00 mm to (116.7, 133.7), turned to 90 degrees
- moved Y3 6.00 mm to (116.7, 145.7), turned to 90 degrees
- moved J1 2.65 mm to (122.7, 121.6)
- moved U10 1.83 mm to (108.9, 113.4), turned to -90 degrees
- moved C33 1.73 mm to (111.3, 119.1)
- moved L2 1.59 mm to (80.2, 84.5), turned to -90 degrees
- moved C32 1.09 mm to (118.3, 110.3)
- moved L1 0.90 mm to (119.8, 84.7), turned to -90 degrees
- moved C23 0.58 mm to (106.3, 119.0)
- moved P16 0.50 mm to (123.0, 138.4)
- moved P6 0.50 mm to (123.0, 141.0)
- moved P15 0.36 mm to (122.5, 155.3)
- moved P7 0.36 mm to (122.5, 152.8)
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Connections:
- C29 pad 2: Net-(Y7-Pad3) -> Net-(C29-Pad2)
- C30 pad 1: Net-(U10-Pad4) -> Net-(C30-Pad1)
- C32 pad 2: Net-(U10-Pad13) -> Net-(C32-Pad2)
- P15 pad 1: Net-(U12-Pad10) -> Net-(P15-Pad1)
- P6 pad 1: Net-(Y7-Pad3) -> Net-(C29-Pad2)
- P7 pad 1: Net-(U12-Pad14) -> Net-(P7-Pad1)
- U10 pad 1: GND -> TXD
- U10 pad 13: Net-(U10-Pad13) -> unconnected-(U10-Pad13)
- U10 pad 15: unconnected-(U10-Pad15) -> D+
- U10 pad 16: VCC -> D-
- U10 pad 2: Net-(U10-Pad2) -> Net-(C32-Pad2)
- U10 pad 3: Net-(U10-Pad3) -> unconnected-(U10-Pad3)
- U10 pad 4: Net-(U10-Pad4) -> VCC
- U10 pad 5: D+ -> RXD
- U10 pad 6: D- -> unconnected-(U10-Pad6)
- U10 pad 7: Net-(U10-Pad7) -> GND
- U10 pad 8: Net-(U10-Pad8) -> (no net)
- U12 pad 10: Net-(U12-Pad10) -> Net-(P15-Pad1)
- U12 pad 14: Net-(U12-Pad14) -> Net-(P7-Pad1)
Routing:
- net Net-(P7-Pad1): track 0.00 -> 36.4 mm, vias 0 -> 2
- net Net-(U12-Pad14): track 35.7 -> 0.00 mm, vias 2 -> 0
- net Net-(P15-Pad1): track 0.00 -> 27.3 mm, vias 0 -> 4
- net Net-(U12-Pad10): track 27.2 -> 0.00 mm, vias 4 -> 0
- net Net-(U10-Pad7): track 26.1 -> 0.00 mm, vias 2 -> 0
- net Net-(U10-Pad22): track 0.00 -> 21.5 mm
- net Net-(U10-Pad23): track 0.00 -> 18.2 mm
- net Net-(C29-Pad2): track 0.00 -> 17.9 mm, vias 0 -> 4
- net Net-(C32-Pad2): track 0.00 -> 17.6 mm
- net Net-(U10-Pad8): track 16.6 -> 0.00 mm
- net Net-(U10-Pad13): track 14.4 -> 0.00 mm
- net Net-(Y7-Pad3): track 13.6 -> 0.00 mm
- net Net-(U10-Pad4): track 9.09 -> 0.00 mm
- net D+: track 20.1 -> 11.4 mm, vias 4 -> 2
- net D-: track 20.0 -> 12.3 mm, vias 2 -> 0
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- added copper zone on B.Cu, net Net-(C29-Pad2)
- added copper zone on F.Cu, net Net-(C29-Pad2)
- added copper zone on F.Cu, net Net-(P15-Pad1)
- added copper zone on B.Cu, net Net-(P7-Pad1)
- removed copper zone on F.Cu, net Net-(U12-Pad10)
- removed copper zone on B.Cu, net Net-(U12-Pad14)
- removed copper zone on B.Cu, net Net-(Y7-Pad3)
- removed copper zone on F.Cu, net unconnected-(Y7-Pad2)
Other:
- board text added: "OpenTheremin V4.2"
- board text removed: "OpenTheremin V4"
